File: hw/metric-gauge/metric-gauge.kicad_pcb (KiCad board)
At the start: 2 copper layers, 86.4 x 48.3 mm, 11 parts, among them J1 Conn_01x02_Socket

Commit message: Update hardware PCB layout and firmware imports
- Relocate mounting holes and update board footprint U2
- Regenerate gerber files
- Import ConstStaticCell in main and remove unused MaybeUninit in http
  module
Parts:
- moved H7 14.0 mm to (82.5, 114.3)
- moved H8 14.0 mm to (158.8, 114.3)
Changed lines of the file:
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@@
 	(footprint "MountingHole:MountingHole_2.1mm"
 		(layer "F.Cu")
-		(at 158.75 100.33)
+		(at 158.75 114.3)
 		(descr "Mounting Hole 2.1mm, no annular, generated by kicad-footprint-generator mountinghole.py")
 		(tags "mountinghole")
@@
 	(footprint "MountingHole:MountingHole_2.1mm"
 		(layer "F.Cu")
-		(at 82.55 100.33)
+		(at 82.55 114.3)
 		(descr "Mounting Hole 2.1mm, no annular, generated by kicad-footprint-generator mountinghole.py")
 		(tags "mountinghole")
